File: eagle/CR78-HB.brd (EAGLE design)
At the start: 100 x 80 mm, 35 parts, among them Q1 2N3904, Q2 2N3904, Q3 2N3904

Commit message: routed with pot change resistor value
Parts:
- R12: value 500R -> 10k
- R20: value 15k -> 526R
Connections:
- net N$8: no longer R12.3
Routing:
- net N$8: track 19.7 -> 14.9 mm
Changed lines of the file:
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@@
 <element name="R10" library="rcl" package="0207/7" value="1M5" x="53.34" y="22.86" rot="R180"/>
 <element name="R11" library="rcl" package="0207/7" value="10k" x="60.833" y="23.622" rot="R270"/>
-<element name="R12" library="pot" package="3RP/1610N" value="500R" x="56.515" y="3.81"/>
+<element name="R12" library="pot" package="3RP/1610N" value="10k" x="56.515" y="3.81"/>
 <element name="R7" library="pot" package="3RP/1610N" value="10KB" x="27.94" y="3.81"/>
 <element name="R19" library="rcl" package="0207/5V" value="10k" x="56.515" y="10.795" rot="R180"/>
@@
 <attribute name="OC_NEWARK" value="38C0355" x="12.7" y="5.08" size="1.778" layer="27" display="off"/>
 </element>
-<element name="R20" library="rcl" package="0207/5V" value="15k" x="45.72" y="6.985" rot="R90"/>
+<element name="R20" library="rcl" package="0207/5V" value="526R" x="45.72" y="6.985" rot="R90"/>
 </elements>
 <signals>
@@
 </signal>
 <signal name="N$8">
-<contactref element="R12" pad="3"/>
-<contactref element="R13" pad="1"/>
 <contactref element="R12" pad="2"/>
 <contactref element="R20" pad="2"/>
 <wire x1="47.625" y1="9.525" x2="45.72" y2="9.525" width="0.8128" layer="16"/>
-<wire x1="50.165" y1="10.795" x2="49.53" y2="10.16" width="0.8128" layer="16"/>
 <wire x1="49.53" y1="10.16" x2="47.625" y2="9.525" width="0.8128" layer="16"/>
-<wire x1="61.515" y1="3.81" x2="57.15" y2="3.81" width="0.8128" layer="16"/>
-<wire x1="57.15" y1="3.81" x2="50.165" y2="10.795" width="0.8128" layer="16"/>
 <wire x1="57.15" y1="3.81" x2="56.515" y2="3.81" width="0.8128" layer="16"/>
+<contactref element="R13" pad="1"/>
+<wire x1="56.515" y1="3.81" x2="50.165" y2="10.795" width="0.8128" layer="16"/>
+<wire x1="49.53" y1="10.16" x2="50.165" y2="10.795" width="0.8128" layer="16"/>
 </signal>
 <signal name="N$9">
@@
 <contactref element="R12" pad="1"/>
 <contactref element="Q2" pad="3"/>
-<contactref element="R20" pad="1"/>
-<wire x1="50.8" y1="3.175" x2="45.72" y2="4.445" width="0.8128" layer="16"/>
-<wire x1="51.435" y1="3.81" x2="50.8" y2="3.175" width="0.8128" layer="16"/>
+<wire x1="51.435" y1="3.81" x2="51.1175" y2="3.4925" width="0.8128" layer="16"/>
+<wire x1="51.1175" y1="3.4925" x2="50.8" y2="3.175" width="0.8128" layer="16"/>
 <wire x1="51.435" y1="3.81" x2="51.515" y2="3.81" width="0.8128" layer="16"/>
 <wire x1="53.34" y1="17.145" x2="51.435" y2="20.32" width="0.8128" layer="16"/>
@@
 <wire x1="45.085" y1="12.065" x2="43.688" y2="10.668" width="0.8128" layer="16"/>
 <wire x1="43.688" y1="10.668" x2="43.688" y2="6.858" width="0.8128" layer="16"/>
+<contactref element="R20" pad="1"/>
 <wire x1="43.688" y1="6.858" x2="45.72" y2="4.445" width="0.8128" layer="16"/>
+<wire x1="45.72" y1="4.445" x2="51.1175" y2="3.4925" width="0.8128" layer="16"/>
 </signal>
 <signal name="N$14">
@@
 <wire x1="80.264" y1="17.526" x2="75.184" y2="23.876" width="0.8128" layer="16"/>
 <wire x1="75.184" y1="23.876" x2="71.628" y2="28.956" width="0.8128" layer="16"/>
-<wire x1="71.628" y1="28.956" x2="12.192" y2="28.956" width="0.8128" layer="16"/>
-<wire x1="12.192" y1="28.956" x2="5.588" y2="22.098" width="0.8128" layer="16"/>
-<wire x1="5.588" y1="22.098" x2="5.588" y2="5.588" width="0.8128" layer="16"/>
+<wire x1="71.628" y1="28.956" x2="11.938" y2="28.956" width="0.8128" layer="16"/>
+<wire x1="11.938" y1="28.956" x2="5.588" y2="22.352" width="0.8128" layer="16"/>
+<wire x1="5.588" y1="22.352" x2="5.588" y2="5.588" width="0.8128" layer="16"/>
 <wire x1="5.588" y1="5.588" x2="7.62" y2="2.54" width="0.8128" layer="16"/>
 <wire x1="7.62" y1="2.54" x2="15.24" y2="2.54" width="0.8128" layer="16"/>

Commit message: cutout
Parts:
- moved Q3 0.72 mm to (69.7, 14.7)
- moved Q2 0.57 mm to (54.1, 17.4)
- moved R17 0.57 mm to (66.9, 26.8)
- moved C7 0.51 mm to (65.3, 15.2)
- moved C2 0.51 mm to (32.3, 14.0)
- moved R8 0.36 mm to (35.2, 14.9)
- moved R13 0.36 mm to (49.9, 14.4)
- moved R16 0.25 mm to (66.9, 24.1)
- moved R4 0.25 mm to (26.7, 14.2)
- moved R5 0.25 mm to (29.2, 14.2)
Routing:
- net GND: track 149.6 -> 148.8 mm
- net N$18: track 31.5 -> 32.2 mm
Other:
- board size 100 x 80 mm -> 100 x 80.8 mm
