File: eagle/CR78-HB.brd (EAGLE design)
At the start: 100 x 80.8 mm, 35 parts, among them Q1 2N3904, Q2 2N3904, Q3 2N3904

Commit message: values for LC
Parts:
- C2: value 82n -> 22n
- C3: value 82n -> 27n
- C4, C5: value 68n -> 22n
- C6: value 27n -> 10n
- R14: value 18k -> 560k
- R19: value 10k -> OMIT
- R4: value 150k -> 390k
Changed lines of the file:
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@@
 <elements>
 <element name="C1" library="rcl" package="C050-025X075" value="27n" x="24.13" y="22.86"/>
-<element name="C2" library="rcl" package="C050-025X075" value="82n" x="32.258" y="13.97" rot="R270"/>
-<element name="C3" library="rcl" package="C050-025X075" value="82n" x="40.64" y="18.415"/>
-<element name="C4" library="rcl" package="C050-025X075" value="68n" x="40.513" y="15.24"/>
-<element name="C5" library="rcl" package="C050-025X075" value="68n" x="43.815" y="22.225"/>
-<element name="C6" library="rcl" package="C050-025X075" value="27n" x="58.42" y="17.78" rot="R270"/>
+<element name="C2" library="rcl" package="C050-025X075" value="22n" x="32.258" y="13.97" rot="R270"/>
+<element name="C3" library="rcl" package="C050-025X075" value="27n" x="40.64" y="18.415"/>
+<element name="C4" library="rcl" package="C050-025X075" value="22n" x="40.513" y="15.24"/>
+<element name="C5" library="rcl" package="C050-025X075" value="22n" x="43.815" y="22.225"/>
+<element name="C6" library="rcl" package="C050-025X075" value="10n" x="58.42" y="17.78" rot="R270"/>
 <element name="C7" library="rcl" package="C050-025X075" value="473" x="65.278" y="15.24" rot="R90"/>
 <element name="C8" library="rcl" package="C050-025X075" value="47p" x="66.04" y="20.955"/>
@@
 <element name="Q3" library="808_lt" package="TO92" value="2N3904" x="69.723" y="14.732" rot="R90"/>
 <element name="R3" library="rcl" package="0207/7" value="270k" x="33.655" y="22.86"/>
-<element name="R14" library="rcl" package="0207/7" value="18k" x="62.23" y="13.97" rot="R90"/>
+<element name="R14" library="rcl" package="0207/7" value="560k" x="62.23" y="13.97" rot="R90"/>
 <element name="R16" library="rcl" package="0207/7" value="470k" x="66.929" y="24.13"/>
 <element name="R17" library="rcl" package="0207/7" value="47k" x="66.929" y="26.797" rot="R180"/>
 <element name="R18" library="rcl" package="0207/7" value="220R" x="68.58" y="6.35" rot="R270"/>
 <element name="R15" library="rcl" package="0207/7" value="100k" x="38.735" y="25.4" rot="R180"/>
-<element name="R4" library="rcl" package="0207/7" value="150k" x="26.67" y="14.224" rot="R270"/>
+<element name="R4" library="rcl" package="0207/7" value="390k" x="26.67" y="14.224" rot="R270"/>
 <element name="R6" library="rcl" package="0207/7" value="56k" x="19.05" y="10.414"/>
 <element name="R2" library="rcl" package="0207/7" value="10k" x="17.78" y="15.24"/>
@@
 <element name="R12" library="pot" package="3RP/1610N" value="10k" x="56.515" y="3.81"/>
 <element name="R7" library="pot" package="3RP/1610N" value="10KB" x="27.94" y="3.81"/>
-<element name="R19" library="rcl" package="0207/5V" value="10k" x="56.515" y="10.795" rot="R180"/>
+<element name="R19" library="rcl" package="0207/5V" value="OMIT" x="56.515" y="10.795" rot="R180"/>
 <element name="BD" library="con-molex" package="22-23-2041" value="22-23-2041" x="12.7" y="5.08">
 <attribute name="MPN" value="22-23-2041" x="12.7" y="5.08" size="1.778" layer="27" display="off"/>

Commit message: values for LB
Parts:
- C2, C4: value 22n -> 12n
- C3: value 27n -> 18n
- C5: value 22n -> 10n
- C6: value 10n -> 8n2
- R14: value 560k -> 680k
Changed lines of the file:
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@@
 <elements>
 <element name="C1" library="rcl" package="C050-025X075" value="27n" x="24.13" y="22.86"/>
-<element name="C2" library="rcl" package="C050-025X075" value="22n" x="32.258" y="13.97" rot="R270"/>
-<element name="C3" library="rcl" package="C050-025X075" value="27n" x="40.64" y="18.415"/>
-<element name="C4" library="rcl" package="C050-025X075" value="22n" x="40.513" y="15.24"/>
-<element name="C5" library="rcl" package="C050-025X075" value="22n" x="43.815" y="22.225"/>
-<element name="C6" library="rcl" package="C050-025X075" value="10n" x="58.42" y="17.78" rot="R270"/>
+<element name="C2" library="rcl" package="C050-025X075" value="12n" x="32.258" y="13.97" rot="R270"/>
+<element name="C3" library="rcl" package="C050-025X075" value="18n" x="40.64" y="18.415"/>
+<element name="C4" library="rcl" package="C050-025X075" value="12n" x="40.513" y="15.24"/>
+<element name="C5" library="rcl" package="C050-025X075" value="10n" x="43.815" y="22.225"/>
+<element name="C6" library="rcl" package="C050-025X075" value="8n2" x="58.42" y="17.78" rot="R270"/>
 <element name="C7" library="rcl" package="C050-025X075" value="473" x="65.278" y="15.24" rot="R90"/>
 <element name="C8" library="rcl" package="C050-025X075" value="47p" x="66.04" y="20.955"/>
@@
 <element name="Q3" library="808_lt" package="TO92" value="2N3904" x="69.723" y="14.732" rot="R90"/>
 <element name="R3" library="rcl" package="0207/7" value="270k" x="33.655" y="22.86"/>
-<element name="R14" library="rcl" package="0207/7" value="560k" x="62.23" y="13.97" rot="R90"/>
+<element name="R14" library="rcl" package="0207/7" value="680k" x="62.23" y="13.97" rot="R90"/>
 <element name="R16" library="rcl" package="0207/7" value="470k" x="66.929" y="24.13"/>
 <element name="R17" library="rcl" package="0207/7" value="47k" x="66.929" y="26.797" rot="R180"/>

Commit message: values for HB
Parts:
- C2: value 12n -> 8n2
- C3: value 18n -> 8n2
- C4: value 12n -> 6n8
- C5: value 10n -> 6n8
- C6: value 8n2 -> 2n2
- R14: value 680k -> 1M5
Changed lines of the file:
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@@
 <elements>
 <element name="C1" library="rcl" package="C050-025X075" value="27n" x="24.13" y="22.86"/>
-<element name="C2" library="rcl" package="C050-025X075" value="12n" x="32.258" y="13.97" rot="R270"/>
-<element name="C3" library="rcl" package="C050-025X075" value="18n" x="40.64" y="18.415"/>
-<element name="C4" library="rcl" package="C050-025X075" value="12n" x="40.513" y="15.24"/>
-<element name="C5" library="rcl" package="C050-025X075" value="10n" x="43.815" y="22.225"/>
-<element name="C6" library="rcl" package="C050-025X075" value="8n2" x="58.42" y="17.78" rot="R270"/>
+<element name="C2" library="rcl" package="C050-025X075" value="8n2" x="32.258" y="13.97" rot="R270"/>
+<element name="C3" library="rcl" package="C050-025X075" value="8n2" x="40.64" y="18.415"/>
+<element name="C4" library="rcl" package="C050-025X075" value="6n8" x="40.513" y="15.24"/>
+<element name="C5" library="rcl" package="C050-025X075" value="6n8" x="43.815" y="22.225"/>
+<element name="C6" library="rcl" package="C050-025X075" value="2n2" x="58.42" y="17.78" rot="R270"/>
 <element name="C7" library="rcl" package="C050-025X075" value="473" x="65.278" y="15.24" rot="R90"/>
 <element name="C8" library="rcl" package="C050-025X075" value="47p" x="66.04" y="20.955"/>
@@
 <element name="Q3" library="808_lt" package="TO92" value="2N3904" x="69.723" y="14.732" rot="R90"/>
 <element name="R3" library="rcl" package="0207/7" value="270k" x="33.655" y="22.86"/>
-<element name="R14" library="rcl" package="0207/7" value="680k" x="62.23" y="13.97" rot="R90"/>
+<element name="R14" library="rcl" package="0207/7" value="1M5" x="62.23" y="13.97" rot="R90"/>
 <element name="R16" library="rcl" package="0207/7" value="470k" x="66.929" y="24.13"/>
 <element name="R17" library="rcl" package="0207/7" value="47k" x="66.929" y="26.797" rot="R180"/>
